File: PCB/PiicoDev-Expansion-Board-for-Raspberry-Pi-Pico.kicad_pcb (KiCad board)
At the start: 2 copper layers, 50.4 x 51.4 mm, 26 parts, among them J1 PiicoDev, J2 JST PH, J3 , J4 , Q1 DMG3415U-7, U1 MCP73832-2-OT

Commit message: Change LED Resistor from 1k to 4.7k
Parts:
- R2: value 1k -> 4k7
