File: PCB/PiicoDev-LiPo-Expansion-Board-for-Raspberry-Pi-Pico.kicad_sch (KiCad schematic)
At the start: 26 parts, among them J1 PiicoDev, J2 JST PH, J3 , J4 , Q1 P-ch MOSFET, U1 LIPO CHARGER

Commit message: update schematic title block
Other:
- title: Expansion Board for Raspberry Pi Pico -> PiicoDev LiPo Expansion Board for Raspberry Pi Pico
Changed lines of the file:
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@@
   (paper "A4")
   (title_block
-    (title "Expansion Board for Raspberry Pi Pico")
+    (title "PiicoDev LiPo Expansion Board for Raspberry Pi Pico")
     (date "2021-10-29")
     (rev "v11")
